Commit message: working sim
no rotation lock and no collision the hight is locked. the size of the grid is wrong thought

File: urdf/sentry.urdf.xacro (robot description, xacro)
@@ -2,10 +2,4 @@
 <!--URDF generated by ONSHAPE BY PTC INC, 1.217-->
 <robot name="sentry_pkg">
-  <!-- "world" is anchor for the planar_x/planar_y/root joint chain below.
-       gz-sim recognizes "world" as the static world frame by name even
-       without this declaration, but strict URDF parsers (e.g. the one
-       robot_state_publisher uses) require every joint's parent link to
-       actually be declared, so it's declared explicitly here too. -->
-  <link name="world"/>
   <link name="body">
     <inertial>
@@ -23,16 +17,4 @@
       </material>
     </visual>
-    <collision>
-      <!-- Body.stl's actual footprint is ~0.595m x 0.595m x 0.252m tall
-           (measured from the mesh); the previous collision cylinder here
-           was radius 0.03 (3cm), ~10x too small, basically a single
-           point contact instead of the real base. That gave the sim
-           robot almost no resistance to tipping under any lateral push
-           (e.g. from cmd_vel). Sized/centered to match the real mesh. -->
-      <origin xyz="0 0 0.1262" rpy="0 0 0"/>
-      <geometry>
-        <cylinder radius="0.28" length="0.252"/>
-      </geometry>
-    </collision>
   </link>
   <link name="head">
@@ -51,10 +33,4 @@
       </material>
     </visual>
-    <collision>
-      <origin xyz="-0.00211769 -0.00164536 0.0741316" rpy="0 -0 1.18195"/>
-      <geometry>
-        <box size="0.2 0.14 0.16075"/>
-      </geometry>
-    </collision>
   </link>
   <link name="lidar">
@@ -89,10 +65,4 @@
       </material>
     </visual>
-    <collision>
-      <origin xyz="0 0 0" rpy="1.5707 0 0"/>
-      <geometry>
-        <cylinder radius="0.024" length="0.018"/>
-      </geometry>
-    </collision>
   </link>
   <link name="odowheel_1">
@@ -111,123 +81,35 @@
       </material>
     </visual>
-    <collision>
-      <origin xyz="0 0 0" rpy="1.5707 0 0"/>
-      <geometry>
-        <cylinder radius="0.024" length="0.018"/>
-      </geometry>
-    </collision>
-  </link>
-  <!-- Constrains the whole chassis to X/Y translation + yaw only, no roll
-       or pitch, by connecting it to the world through two prismatic joints
-       and one revolute (yaw) joint instead of leaving it a free 6DOF body.
-       Movement is already purely commanded (VelocityControl), not derived
-       from real wheel/ground physics, so this loses nothing functionally
-       and makes tipping over on a lip or ramp kinematically impossible
-       (the previous fixes, wider body collision and disabled gravity,
-       reduced how often it tipped but couldn't eliminate it; a ramp's
-       inclined surface can still impart roll/pitch torque on a free body
-       no matter how wide its footprint is). Mirrors what the real robot's
-       suspension does: isolates the chassis from ground-level disturbances. -->
-  <link name="planar_x">
-    <inertial>
-      <!-- Deliberately not near-zero (an earlier version used mass 0.0001 /
-           inertia 1e-9): confirmed empirically that made the yaw joint spin
-           itself up to its velocity limit under a corner collision with 0
-           commanded velocity and 0 reported effort, i.e. not driven by any
-           controller; a near-massless connector link between joints is a
-           known DART/ODE instability under contact (any small residual
-           constraint force produces huge spurious acceleration on a link
-           with almost no inertia to resist it). Still tiny relative to the
-           real chassis (mass 0.05, izz 0.00226) so it doesn't meaningfully
-           change commanded motion, just gives the solver something
-           non-degenerate to work with. -->
-      <mass value="0.05"/>
-      <origin xyz="0 0 0" rpy="0 0 0"/>
-      <inertia ixx="1e-4" ixy="0" ixz="0" iyy="1e-4" iyz="0" izz="1e-4"/>
-    </inertial>
-  </link>
-  <joint name="world_to_planar_x" type="prismatic">
-    <parent link="world"/>
-    <child link="planar_x"/>
-    <axis xyz="1 0 0"/>
-    <limit lower="-1000" upper="1000" effort="1000" velocity="10"/>
-  </joint>
-  <link name="planar_y">
-    <inertial>
-      <!-- Deliberately not near-zero (an earlier version used mass 0.0001 /
-           inertia 1e-9): confirmed empirically that made the yaw joint spin
-           itself up to its velocity limit under a corner collision with 0
-           commanded velocity and 0 reported effort, i.e. not driven by any
-           controller; a near-massless connector link between joints is a
-           known DART/ODE instability under contact (any small residual
-           constraint force produces huge spurious acceleration on a link
-           with almost no inertia to resist it). Still tiny relative to the
-           real chassis (mass 0.05, izz 0.00226) so it doesn't meaningfully
-           change commanded motion, just gives the solver something
-           non-degenerate to work with. -->
-      <mass value="0.05"/>
-      <origin xyz="0 0 0" rpy="0 0 0"/>
-      <inertia ixx="1e-4" ixy="0" ixz="0" iyy="1e-4" iyz="0" izz="1e-4"/>
-    </inertial>
-  </link>
-  <joint name="planar_x_to_y" type="prismatic">
-    <parent link="planar_x"/>
-    <child link="planar_y"/>
-    <axis xyz="0 1 0"/>
-    <limit lower="-1000" upper="1000" effort="1000" velocity="10"/>
-  </joint>
-  <link name="yaw_base">
-    <inertial>
-      <!-- Deliberately not near-zero (an earlier version used mass 0.0001 /
-           inertia 1e-9): confirmed empirically that made the yaw joint spin
-           itself up to its velocity limit under a corner collision with 0
-           commanded velocity and 0 reported effort, i.e. not driven by any
-           controller; a near-massless connector link between joints is a
-           known DART/ODE instability under contact (any small residual
-           constraint force produces huge spurious acceleration on a link
-           with almost no inertia to resist it). Still tiny relative to the
-           real chassis (mass 0.05, izz 0.00226) so it doesn't meaningfully
-           change commanded motion, just gives the solver something
-           non-degenerate to work with. -->
-      <mass value="0.05"/>
-      <origin xyz="0 0 0" rpy="0 0 0"/>
-      <inertia ixx="1e-4" ixy="0" ixz="0" iyy="1e-4" iyz="0" izz="1e-4"/>
-    </inertial>
-  </link>
-  <joint name="planar_y_to_root_yaw" type="continuous">
-    <parent link="planar_y"/>
-    <child link="yaw_base"/>
-    <axis xyz="0 0 1"/>
-    <limit effort="1000" velocity="10"/>
-    <!-- Without damping, a corner collision's reaction torque spins this
-         joint up and it never slows back down on its own (confirmed: caught
-         it pegged at its 10 rad/s velocity limit with 0 effort reported,
-         i.e. not driven by the controller at all, purely leftover momentum);
-         explorer never commands yaw, but once spinning like that it kept
-         dragging/fighting the wall it was wedged against by friction,
-         reads as "stuck no matter what heading is picked" even though X/Y
-         are independently commandable. suspension_z already had damping for
-         the same reason; this joint was missed. -->
-    <dynamics damping="20.0"/>
-  </joint>
-  <!-- X/Y/yaw above are driven (JointController), always exactly what's
-       commanded. Z is the only passive/gravity-driven DOF: lets the
-       chassis ride up over a ramp or lip instead of being pinned to a
-       fixed height, without needing roll/pitch to do it (root stays flat;
-       it rises onto a ramp rather than tilting to match its slope).
-       Simplified from an earlier 3-joint suspension (Z + roll + pitch)
-       that also let the chassis tilt; more physically faithful, but
-       more tuning surface than needed here, since roll/pitch was only
-       ever needed to prevent flipping, and Z alone already makes that
-       impossible (no roll/pitch DOF exists at all now, not just a limited
-       one) while being simpler to reason about. -->
-  <link name="root"/>
-  <joint name="suspension_z" type="prismatic">
-    <parent link="yaw_base"/>
-    <child link="root"/>
-    <axis xyz="0 0 1"/>
-    <limit lower="-0.3" upper="0.3" effort="1000" velocity="5"/>
-    <dynamics damping="5.0"/>
-  </joint>
+  </link>
+  <!-- root is a genuinely free 6DOF body again, with no collision anywhere
+       on the model (see body/head/odowheel above), and no parent joint at
+       all, it's the URDF's implicit base link.
+       This is a deliberate reversal of an earlier design that constrained
+       root through a world->px->root chain of translation-only prismatic
+       joints specifically to make rotation structurally impossible (real
+       chassis is holonomic and never turns) and prevent wall-contact
+       torque from flipping it. That design blocked true teleporting: gz's
+       physics only honors a direct world-pose write (the "set_pose"
+       service sim/auto_explore.py needs for its grid sweep) on a link
+       gz-physics' FreeGroup API recognizes as free-floating, and a link
+       with a parent joint doesn't qualify, confirmed empirically,
+       set_pose calls against the old jointed root silently no-op'd.
+       Free + collision-free removes both problems at once: nothing (no
+       contact) can ever apply the torque the old design was defending
+       against, so root can't actually flip even though rotation is
+       physically possible again, and gz now treats it as a normal
+       free body that set_pose actually moves.
+       Since root is the base link again (as it was before the joint-chain
+       design), robot_state_publisher has nothing to publish world->root
+       from on its own, sentry_pkg/launch/auto.launch.py's default
+       (publish_odom_tf:=true, odom_frame:=odom) is what supplies that via
+       odom_to_tf, same as real hardware; no override needed. -->
+  <link name="root">
+    <inertial>
+      <mass value="0.0507536"/>
+      <origin xyz="-2.33205e-05 -3.02404e-05 0.160359" rpy="0 -0 0"/>
+      <inertia ixx="0.00226416" ixy="0" ixz="0" iyy="0.00226416" iyz="0" izz="0.00226416"/>
+    </inertial>
+  </link>
   <joint name="fastened_2" type="fixed">
     <origin xyz="0 0 0" rpy="0 -0 3.14159"/>
@@ -260,11 +142,22 @@
     <child link="odowheel_1"/>
   </joint>
-  <!-- Gravity is left ON here (unlike an earlier attempt that disabled it):
-       the suspension_z joint above needs gravity + normal contact force
-       to naturally settle the chassis onto the floor/ramp at the correct
-       height, the same way a real suspended vehicle does. Disabling
-       gravity made the robot immune to floor lips but also unable to
-       climb ramps at all, since a chassis with no weight has nothing
-       pressing it down to follow the ground's shape. -->
+  <!-- Gravity is off on every link: root is genuinely free-floating now
+       (see the link definition above) with no collision to rest on
+       anything, so gravity would otherwise just make it fall forever. -->
+  <gazebo reference="root">
+    <gravity>false</gravity>
+  </gazebo>
+  <gazebo reference="body">
+    <gravity>false</gravity>
+  </gazebo>
+  <gazebo reference="head">
+    <gravity>false</gravity>
+  </gazebo>
+  <gazebo reference="odowheel">
+    <gravity>false</gravity>
+  </gazebo>
+  <gazebo reference="odowheel_1">
+    <gravity>false</gravity>
+  </gazebo>
   <gazebo reference="lidar">
     <sensor name="lidar" type="gpu_lidar">
@@ -285,5 +178,5 @@
         <range>
           <!-- Matches RPLIDAR A2M8 datasheet: 0.15-12m -->
-          <min>0.15</min>
+          <min>0.2</min>
           <max>12.0</max>
           <resolution>0.015000</resolution>
@@ -311,30 +204,4 @@
       <joint_name>odowheel_x</joint_name>
       <joint_name>odowheel_y</joint_name>
-      <!-- OdometryPublisher's /odom orientation reads identity regardless
-           of root's actual yaw now that root is joint-constrained (verified:
-           the physics engine's own ground truth for root's link pose DOES
-           show correct rotation, but OdometryPublisher's ROS-facing output
-           doesn't reflect it; some assumption of the plugin's about a
-           freely-floating base no longer holds). This joint's own position
-           IS the robot's yaw by construction, so it's tracked here and
-           sentry_pkg's odom_to_tf node uses it directly instead of trusting
-           /odom's orientation field. -->
-      <joint_name>planar_y_to_root_yaw</joint_name>
-      <!-- Same story, but for Y position instead of yaw: confirmed via
-           /world/.../pose/info and /world/.../state that root's Y position
-           genuinely does update in the physics engine when
-           planar_x_to_y is driven, but /odom's Y field stays 0 regardless.
-           X position, oddly, reports correctly through /odom (only Y and
-           yaw are affected); tracked here as a further workaround so
-           odom_to_tf can source Y from here too instead of /odom. -->
-      <joint_name>planar_x_to_y</joint_name>
-      <!-- robot_state_publisher needs /joint_states data for every
-           non-fixed joint to compute a single connected TF tree; any
-           untracked joint (world_to_planar_x and the 3 suspension joints
-           below were missing) fragments the tree into unconnected pieces,
-           breaking TF lookups like root->lidar entirely (not just reporting
-           a wrong value, the frames don't connect at all). -->
-      <joint_name>world_to_planar_x</joint_name>
-      <joint_name>suspension_z</joint_name>
       <ros>
         <argument>-p use_sim_time:=true</argument>
@@ -364,52 +231,20 @@
       <cmd_min>-5</cmd_min>
     </plugin>
-    <!-- Lets the chassis actually be driven around in sim (e.g. to sweep
-         the room for mapping). Real hardware moves via the DJI Type-C board
+    <!-- Lets the chassis actually be driven around in sim manually (e.g.
+         sim/wasd_teleop.py). Real hardware moves via the DJI Type-C board
          directly, not ROS, so this only exists for sim; there's no
          equivalent on the real robot.
-         VelocityControl (which set a free body's velocity directly) can't
-         be used anymore now that root is joint-constrained rather than a
-         free 6DOF body; confirmed empirically, it produced zero motion
-         when targeted at "root" since root has no linear DOF of its own
-         (only the yaw joint). Driving a joint-constrained base needs
-         per-joint velocity control instead, one JointController per DOF;
-         sim/sim/cmd_vel_to_joints.py splits a single /cmd_vel Twist into
-         the 3 per-joint velocity topics these subscribe to. -->
-    <!-- use_force_commands=false (direct kinematic velocity injection)
-         silently fails to move planar_x_to_y specifically: confirmed
-         empirically that world_to_planar_x (parent="world", fixed) and
-         planar_y_to_root_yaw (parent="planar_y", not itself kinematically
-         driven) both work fine in kinematic mode, but planar_x_to_y's
-         parent (planar_x) is itself the output link of another
-         kinematically-controlled joint, and gz-sim's kinematic velocity
-         mode doesn't compose across that chaining. Switched all three to
-         force/PID mode so motion propagates through normal physics
-         integration instead. -->
-    <plugin filename="ignition-gazebo-joint-controller-system" name="ignition::gazebo::systems::JointController">
-      <joint_name>world_to_planar_x</joint_name>
-      <use_force_commands>true</use_force_commands>
-      <p_gain>50</p_gain>
-      <i_gain>1</i_gain>
-      <d_gain>0</d_gain>
-      <i_max>10</i_max>
-      <i_min>-10</i_min>
-    </plugin>
-    <plugin filename="ignition-gazebo-joint-controller-system" name="ignition::gazebo::systems::JointController">
-      <joint_name>planar_x_to_y</joint_name>
-      <use_force_commands>true</use_force_commands>
-      <p_gain>50</p_gain>
-      <i_gain>1</i_gain>
-      <d_gain>0</d_gain>
-      <i_max>10</i_max>
-      <i_min>-10</i_min>
-    </plugin>
-    <plugin filename="ignition-gazebo-joint-controller-system" name="ignition::gazebo::systems::JointController">
-      <joint_name>planar_y_to_root_yaw</joint_name>
-      <use_force_commands>true</use_force_commands>
-      <p_gain>50</p_gain>
-      <i_gain>1</i_gain>
-      <d_gain>0</d_gain>
-      <i_max>10</i_max>
-      <i_min>-10</i_min>
+         root is a genuinely free link again (see the link definition
+         above), so unlike the old prismatic-joint-chain design, a single
+         VelocityControl plugin can take a Twist directly instead of
+         needing sim/cmd_vel_to_joints.py to split it across two
+         per-joint JointControllers. angular.z still isn't zeroed out
+         here structurally the way the removed joint chain enforced it
+         (root can physically rotate again, see the link definition
+         above), so it's on wasd_teleop.py/whatever publishes /cmd_vel to
+         not command it, matching the real robot's holonomic,
+         never-turns behavior by convention rather than by construction. -->
+    <plugin filename="ignition-gazebo-velocity-control-system" name="ignition::gazebo::systems::VelocityControl">
+      <topic>/model/sentry/cmd_vel</topic>
     </plugin>
   </gazebo>

Commit message: tunned it
added back direct head control and tunned the auto_explore.py to stay in bounds

File: urdf/sentry.urdf.xacro (robot description, xacro)
@@ -104,10 +104,28 @@
        from on its own, sentry_pkg/launch/auto.launch.py's default
        (publish_odom_tf:=true, odom_frame:=odom) is what supplies that via
-       odom_to_tf, same as real hardware; no override needed. -->
+       odom_to_tf, same as real hardware; no override needed.
+       Rotational inertia (ixx/iyy/izz) is inflated ~1000x past body's
+       real value as a soft rotation lock: even with the active headlink
+       PID removed and auto_explore.py's model_only joint reset before
+       every set_pose (see that file), occasional small chassis rotation
+       was still observed after a teleport, root's own angular velocity
+       isn't part of any joint's state (root has no parent joint), so
+       nothing resets it if a teleport's hard position discontinuity
+       momentarily induces a reaction impulse through headlink/odowheel_x/
+       odowheel_y (all still attached to body, hence root, via real
+       joints). This is the same soft-lock idea an earlier design used
+       before it was replaced with a hard kinematic joint lock (see
+       above), but that lock was defeated by repeated *contact* torque
+       accumulation, which can't happen any more since this model has no
+       collision anywhere; the only remaining torque source is an
+       occasional single-step reaction impulse, and a large rotational
+       inertia suppresses the angular velocity that impulse produces
+       (impulse / inertia) to something negligible without needing any
+       active force control. -->
   <link name="root">
     <inertial>
       <mass value="0.0507536"/>
       <origin xyz="-2.33205e-05 -3.02404e-05 0.160359" rpy="0 -0 0"/>
-      <inertia ixx="0.00226416" ixy="0" ixz="0" iyy="0.00226416" iyz="0" izz="0.00226416"/>
+      <inertia ixx="2.26416" ixy="0" ixz="0" iyy="2.26416" iyz="0" izz="2.26416"/>
     </inertial>
   </link>
@@ -211,6 +229,21 @@
          sim/head_sweep.py, bridged into ROS) drive the head turn: publish a
          target angle (rad) on /model/sentry/joint/headlink/cmd_pos and this
-         PID controller tracks it. Without this plugin nothing can command
-         the head at all.
+         PID controller tracks it.
+         Reintroduced after being removed for a while: this plugin holds
+         its target via continuous PID torque, and since body/root are
+         rigidly fastened with root a genuinely free 6DOF link (no parent
+         joint, see the root link definition above), that reaction torque
+         used to have nowhere to go but into rotating the whole free
+         root/body assembly, which compounded into visible chassis
+         rotation drift over an auto_explore.py sweep and corrupted the
+         map. Safe to bring back now that both of that bug's actual fixes
+         are in place: root's rotational inertia is inflated ~1000x (see
+         the root link definition above), so any reaction torque this PID
+         still produces yields negligible angular velocity, and
+         auto_explore.py's teleport() now resets all joint state
+         (including headlink) via a model_only WorldReset both before AND
+         after every set_pose, so even a transient PID reaction from a
+         teleport's position discontinuity gets wiped before the next hop
+         either way.
          <topic> is set explicitly here (the plugin's own auto-generated
          default is .../headlink/0/cmd_pos) because that "/0/" index segment
