Commit message: Add head pitch joint and simulated RealSense camera to sentry sim
Adds a head_pitch link/joint (independent of the existing yaw-only
headlink) carrying a camera link with an rgbd_camera gz sensor
(D435-like FOV/resolution), wired into the existing JointStatePublisher
and a new JointPositionController alongside headlink's. sim.launch.py
gets matching bridges: /head_pitch_cmd for the new joint, and camera
image/depth/camera_info bridges remapped to the same topic names
realsense-ros uses on real hardware, so realsense-yolov8-nitros-bridge's
CV pipeline can run against sim unmodified.

Placeholder box geometry and mount origin until a real camera mesh and
measured offset exist.

File: urdf/sentry.urdf.xacro (robot description, xacro)
@@ -47,4 +47,32 @@
       <material name="0.615686_0.811765_0.929412_0.000000_0.000000">
         <color rgba="0.615686 0.811765 0.929412 1"/>
+      </material>
+    </visual>
+  </link>
+  <!-- Pitch stage for the head, so a camera mounted on it can tilt
+       independently of the yaw-only headlink joint below. No mesh of its
+       own, just a bare kinematic link the camera is fastened to. -->
+  <link name="head_pitch">
+    <inertial>
+      <mass value="0.005"/>
+      <origin xyz="0 0 0" rpy="0 0 0"/>
+      <inertia ixx="1e-06" ixy="0" ixz="0" iyy="1e-06" iyz="0" izz="1e-06"/>
+    </inertial>
+  </link>
+  <!-- Approximates a RealSense D435 (90x25x25mm, 72g); no mesh exists for
+       it yet so a plain box visual stands in until one is added. -->
+  <link name="camera">
+    <inertial>
+      <mass value="0.072"/>
+      <origin xyz="0 0 0" rpy="0 0 0"/>
+      <inertia ixx="1.05e-05" ixy="0" ixz="0" iyy="5.4e-05" iyz="0" izz="5.4e-05"/>
+    </inertial>
+    <visual>
+      <origin xyz="0 0 0" rpy="0 0 0"/>
+      <geometry>
+        <box size="0.025 0.09 0.025"/>
+      </geometry>
+      <material name="0.1_0.1_0.1_0.000000_0.000000">
+        <color rgba="0.1 0.1 0.1 1"/>
       </material>
     </visual>
@@ -148,4 +176,19 @@
     <child link="lidar"/>
   </joint>
+  <!-- Pitch axis for the head-mounted camera. Placeholder mount point
+       (front-center of head, y-axis tilt) until it's positioned against
+       the real head mesh's geometry. -->
+  <joint name="headpitch" type="revolute">
+    <origin xyz="0.1 0 0" rpy="0 0 0"/>
+    <axis xyz="0 1 0"/>
+    <parent link="head"/>
+    <child link="head_pitch"/>
+    <limit lower="-0.6" upper="0.6" effort="5" velocity="3"/>
+  </joint>
+  <joint name="cameralink" type="fixed">
+    <origin xyz="0 0 0" rpy="0 0 0"/>
+    <parent link="head_pitch"/>
+    <child link="camera"/>
+  </joint>
   <joint name="odowheel_x" type="continuous">
     <origin xyz="-0.089012 -0.009 0.0286405" rpy="3.14159 -0 3.14159"/>
@@ -170,4 +213,10 @@
   </gazebo>
   <gazebo reference="head">
+    <gravity>false</gravity>
+  </gazebo>
+  <gazebo reference="head_pitch">
+    <gravity>false</gravity>
+  </gazebo>
+  <gazebo reference="camera">
     <gravity>false</gravity>
   </gazebo>
@@ -208,4 +257,31 @@
     </sensor>
   </gazebo>
+  <!-- RealSense D435-like RGBD camera for CV testing (yolov8/nitros bridge
+       etc). rgbd_camera bundles color + depth + camera_info under one
+       sensor; <topic> is the prefix each is auto-published under (see
+       sim/launch/sim.launch.py's camera bridges for the full subtopic
+       names and how they're remapped to match realsense-ros' own topic
+       names, so nodes written against real hardware work unmodified here). -->
+  <gazebo reference="camera">
+    <sensor name="camera" type="rgbd_camera">
+      <always_on>true</always_on>
+      <visualize>true</visualize>
+      <update_rate>30</update_rate>
+      <topic>camera</topic>
+      <gz_frame_id>camera</gz_frame_id>
+      <camera>
+        <horizontal_fov>1.5184</horizontal_fov>
+        <image>
+          <width>640</width>
+          <height>480</height>
+          <format>R8G8B8</format>
+        </image>
+        <clip>
+          <near>0.1</near>
+          <far>10.0</far>
+        </clip>
+      </camera>
+    </sensor>
+  </gazebo>
   <gazebo>
     <plugin filename="ignition-gazebo-odometry-publisher-system" name="ignition::gazebo::systems::OdometryPublisher">
@@ -224,4 +300,5 @@
     <plugin filename="ignition-gazebo-joint-state-publisher-system" name="ignition::gazebo::systems::JointStatePublisher">
       <joint_name>headlink</joint_name>
+      <joint_name>headpitch</joint_name>
       <joint_name>odowheel_x</joint_name>
       <joint_name>odowheel_y</joint_name>
@@ -268,4 +345,19 @@
       <cmd_min>-5</cmd_min>
     </plugin>
+    <!-- Same idea as headlink's controller above: publish a target angle
+         (rad, within headpitch's +/-0.6 limit) on
+         /model/sentry/joint/headpitch/cmd_pos and this PID tracks it, so
+         the camera can be tilted from the gz GUI or a bridged ROS topic. -->
+    <plugin filename="ignition-gazebo-joint-position-controller-system" name="ignition::gazebo::systems::JointPositionController">
+      <joint_name>headpitch</joint_name>
+      <topic>/model/sentry/joint/headpitch/cmd_pos</topic>
+      <p_gain>2.0</p_gain>
+      <i_gain>0.1</i_gain>
+      <d_gain>0.05</d_gain>
+      <i_max>1</i_max>
+      <i_min>-1</i_min>
+      <cmd_max>5</cmd_max>
+      <cmd_min>-5</cmd_min>
+    </plugin>
     <!-- Lets the chassis actually be driven around in sim manually (e.g.
          sim/wasd_teleop.py). Real hardware moves via the DJI Type-C board

Commit message: Bump camera to 60Hz and reposition headpitch above the lidar
Real hardware's RealSense runs at 60fps (see
realsense-yolov8-nitros-bridge/config/realsense_640x480x60.yaml), so match
that in sim instead of the placeholder 30Hz. Also moves headpitch's mount
point from an arbitrary front-center placeholder to directly above the
lidar (same x/y as lidarlink, z raised ~5cm to clear it), per feedback
that it should attach to the existing head structure near the lidar.

File: urdf/sentry.urdf.xacro (robot description, xacro)
@@ -176,9 +176,9 @@
     <child link="lidar"/>
   </joint>
-  <!-- Pitch axis for the head-mounted camera. Placeholder mount point
-       (front-center of head, y-axis tilt) until it's positioned against
-       the real head mesh's geometry. -->
+  <!-- Pitch axis for the head-mounted camera. Mounted directly above the
+       lidar (same x/y as lidarlink's origin above, z raised ~5cm to clear
+       it) so the camera looks out from the same face of the head. -->
   <joint name="headpitch" type="revolute">
-    <origin xyz="0.1 0 0" rpy="0 0 0"/>
+    <origin xyz="-0.170562 -0.139254 0.1218" rpy="0 0 0"/>
     <axis xyz="0 1 0"/>
     <parent link="head"/>
@@ -262,10 +262,12 @@
        sim/launch/sim.launch.py's camera bridges for the full subtopic
        names and how they're remapped to match realsense-ros' own topic
-       names, so nodes written against real hardware work unmodified here). -->
+       names, so nodes written against real hardware work unmodified here).
+       60Hz matches real hardware's profile (see
+       realsense-yolov8-nitros-bridge/config/realsense_640x480x60.yaml). -->
   <gazebo reference="camera">
     <sensor name="camera" type="rgbd_camera">
       <always_on>true</always_on>
       <visualize>true</visualize>
-      <update_rate>30</update_rate>
+      <update_rate>60</update_rate>
       <topic>camera</topic>
       <gz_frame_id>camera</gz_frame_id>

Commit message: Center headpitch mount on the head (x/y=0), keep lidar-matched height
Per feedback: x/y should be centered on the head rather than offset to
match the lidar's mount point; only the z height (clearing the lidar)
was correct.

File: urdf/sentry.urdf.xacro (robot description, xacro)
@@ -176,9 +176,8 @@
     <child link="lidar"/>
   </joint>
-  <!-- Pitch axis for the head-mounted camera. Mounted directly above the
-       lidar (same x/y as lidarlink's origin above, z raised ~5cm to clear
-       it) so the camera looks out from the same face of the head. -->
+  <!-- Pitch axis for the head-mounted camera. Centered on the head (x/y=0)
+       at the same height as the lidar's mount z, raised ~5cm to clear it. -->
   <joint name="headpitch" type="revolute">
-    <origin xyz="-0.170562 -0.139254 0.1218" rpy="0 0 0"/>
+    <origin xyz="0 0 0.1218" rpy="0 0 0"/>
     <axis xyz="0 1 0"/>
     <parent link="head"/>

Commit message: Move camera forward on the head (+8cm x)
Per feedback: camera was centered inside the head; shift it forward so
it sits out past the head's front face.

File: urdf/sentry.urdf.xacro (robot description, xacro)
@@ -176,8 +176,10 @@
     <child link="lidar"/>
   </joint>
-  <!-- Pitch axis for the head-mounted camera. Centered on the head (x/y=0)
-       at the same height as the lidar's mount z, raised ~5cm to clear it. -->
+  <!-- Pitch axis for the head-mounted camera. Centered laterally (y=0) at
+       the same height as the lidar's mount z (raised ~5cm to clear it),
+       moved forward (+x) from head center so it sits out past the head's
+       front face rather than buried inside it. -->
   <joint name="headpitch" type="revolute">
-    <origin xyz="0 0 0.1218" rpy="0 0 0"/>
+    <origin xyz="0.08 0 0.1218" rpy="0 0 0"/>
     <axis xyz="0 1 0"/>
     <parent link="head"/>

Commit message: Counter-rotate camera mount to align with head mesh's visual rotation
The camera sat skewed relative to the rendered head because
headpitch's origin used rpy=0 (the link's raw frame) while head's own
<visual> block is rotated rpy="0 0 1.18195". Countering that rotation
on the mount aligns the camera box with the head as actually rendered.

File: urdf/sentry.urdf.xacro (robot description, xacro)
@@ -179,7 +179,10 @@
        the same height as the lidar's mount z (raised ~5cm to clear it),
        moved forward (+x) from head center so it sits out past the head's
-       front face rather than buried inside it. -->
+       front face rather than buried inside it. rpy counters head's own
+       <visual> mesh rotation (rpy="0 0 1.18195") so the camera box sits
+       flush/aligned with the head mesh as rendered instead of skewed
+       relative to it. -->
   <joint name="headpitch" type="revolute">
-    <origin xyz="0.08 0 0.1218" rpy="0 0 0"/>
+    <origin xyz="0.08 0 0.1218" rpy="0 0 -1.18195"/>
     <axis xyz="0 1 0"/>
     <parent link="head"/>

Commit message: Flip camera mount rotation sign (+1.18195 instead of -1.18195)
Previous sign was the wrong direction per feedback.

File: urdf/sentry.urdf.xacro (robot description, xacro)
@@ -179,10 +179,10 @@
        the same height as the lidar's mount z (raised ~5cm to clear it),
        moved forward (+x) from head center so it sits out past the head's
-       front face rather than buried inside it. rpy counters head's own
+       front face rather than buried inside it. rpy matches head's own
        <visual> mesh rotation (rpy="0 0 1.18195") so the camera box sits
        flush/aligned with the head mesh as rendered instead of skewed
        relative to it. -->
   <joint name="headpitch" type="revolute">
-    <origin xyz="0.08 0 0.1218" rpy="0 0 -1.18195"/>
+    <origin xyz="0.08 0 0.1218" rpy="0 0 1.18195"/>
     <axis xyz="0 1 0"/>
     <parent link="head"/>

Commit message: Try rpy z = 1.18195 - pi/2 for camera mount (still tuning)
Previous value (1.18195) was reported exactly 90deg off; trying the
smaller candidate first per feedback, to be confirmed against the live
camera feed once rviz is up.

File: urdf/sentry.urdf.xacro (robot description, xacro)
@@ -179,10 +179,11 @@
        the same height as the lidar's mount z (raised ~5cm to clear it),
        moved forward (+x) from head center so it sits out past the head's
-       front face rather than buried inside it. rpy matches head's own
-       <visual> mesh rotation (rpy="0 0 1.18195") so the camera box sits
-       flush/aligned with the head mesh as rendered instead of skewed
-       relative to it. -->
+       front face rather than buried inside it. rpy z tuned empirically
+       against the rendered scene/camera feed (head's own <visual> mesh
+       rotation is rpy="0 0 1.18195" but that alone overshot by 90deg;
+       this is that value minus pi/2, still being verified against the
+       live feed -- may need further tuning). -->
   <joint name="headpitch" type="revolute">
-    <origin xyz="0.08 0 0.1218" rpy="0 0 1.18195"/>
+    <origin xyz="0.08 0 0.1218" rpy="0 0 -0.38885"/>
     <axis xyz="0 1 0"/>
     <parent link="head"/>

Commit message: Confirm camera mount rotation correct; update comment

File: urdf/sentry.urdf.xacro (robot description, xacro)
@@ -180,8 +180,8 @@
        moved forward (+x) from head center so it sits out past the head's
        front face rather than buried inside it. rpy z tuned empirically
-       against the rendered scene/camera feed (head's own <visual> mesh
-       rotation is rpy="0 0 1.18195" but that alone overshot by 90deg;
-       this is that value minus pi/2, still being verified against the
-       live feed, may need further tuning). -->
+       against the rendered scene/camera feed and confirmed correct
+       (head's own <visual> mesh rotation is rpy="0 0 1.18195", but
+       matching that alone overshot by 90deg; this is that value minus
+       pi/2). -->
   <joint name="headpitch" type="revolute">
     <origin xyz="0.08 0 0.1218" rpy="0 0 -0.38885"/>

Commit message: Rotate camera 180 degrees (lens was facing backwards)

File: urdf/sentry.urdf.xacro (robot description, xacro)
@@ -180,10 +180,10 @@
        moved forward (+x) from head center so it sits out past the head's
        front face rather than buried inside it. rpy z tuned empirically
-       against the rendered scene/camera feed and confirmed correct
-       (head's own <visual> mesh rotation is rpy="0 0 1.18195", but
-       matching that alone overshot by 90deg; this is that value minus
-       pi/2). -->
+       against the rendered scene/camera feed (head's own <visual> mesh
+       rotation is rpy="0 0 1.18195"; this is that value minus pi/2, then
+       rotated a further 180deg per feedback that the lens was facing
+       backwards). -->
   <joint name="headpitch" type="revolute">
-    <origin xyz="0.08 0 0.1218" rpy="0 0 -0.38885"/>
+    <origin xyz="0.08 0 0.1218" rpy="0 0 2.75274"/>
     <axis xyz="0 1 0"/>
     <parent link="head"/>

Commit message: Rotate camera another 180 degrees (back to pre-flip value)

File: urdf/sentry.urdf.xacro (robot description, xacro)
@@ -181,9 +181,9 @@
        front face rather than buried inside it. rpy z tuned empirically
        against the rendered scene/camera feed (head's own <visual> mesh
-       rotation is rpy="0 0 1.18195"; this is that value minus pi/2, then
-       rotated a further 180deg per feedback that the lens was facing
-       backwards). -->
+       rotation is rpy="0 0 1.18195"; this is that value minus pi/2. A
+       subsequent 180deg flip turned out to be wrong too, so this is
+       back to that original value). -->
   <joint name="headpitch" type="revolute">
-    <origin xyz="0.08 0 0.1218" rpy="0 0 2.75274"/>
+    <origin xyz="0.08 0 0.1218" rpy="0 0 -0.38885"/>
     <axis xyz="0 1 0"/>
     <parent link="head"/>

Commit message: Fix ign topic -e stdout buffering in relay; move camera further forward
head_slider_relay: `ign topic -e` fully-buffers stdout when piped (not
a TTY), so without `stdbuf -oL` its lines never reached the relay in
real time. This was masked during testing by an unrelated stale-build
bug (see next paragraph) that made it look like nothing was working at
all.

Camera offset bumped 0.08m -> 0.16m forward. Note: the extended "all
black/flat" image investigation that preceded this turned out to be a
false lead -- the installed sim package had silently fallen back to
copied (non-symlinked) files after a manual `colcon build
--packages-select sim` omitted --symlink-install, so xacro edits
during that window were never actually taking effect on relaunch
regardless of position/sensor-type changes tried. Rebuilding with
--symlink-install (see install-sim.sh, which always includes it)
fixed the live-editing setup; the camera now correctly renders varied
scene content.

File: urdf/sentry.urdf.xacro (robot description, xacro)
@@ -185,5 +185,5 @@
        back to that original value). -->
   <joint name="headpitch" type="revolute">
-    <origin xyz="0.08 0 0.1218" rpy="0 0 -0.38885"/>
+    <origin xyz="0.16 0 0.1218" rpy="0 0 -0.38885"/>
     <axis xyz="0 1 0"/>
     <parent link="head"/>

Commit message: Pull camera back a bit (0.16m -> 0.1m forward offset)

File: urdf/sentry.urdf.xacro (robot description, xacro)
@@ -185,5 +185,5 @@
        back to that original value). -->
   <joint name="headpitch" type="revolute">
-    <origin xyz="0.16 0 0.1218" rpy="0 0 -0.38885"/>
+    <origin xyz="0.1 0 0.1218" rpy="0 0 -0.38885"/>
     <axis xyz="0 1 0"/>
     <parent link="head"/>
