Commit message: Point sim's rviz launch at its own config copy; speed up head movement
Removes the cross-package share_directory lookup into sentry_pkg now
that sim.launch.py owns its own copy of the rviz config. Also raises
headlink/headpitch velocity limits (3 -> 10 rad/s) and shortens
head_sweep.py's sweep period (16s -> 6s), since the joints' own
velocity limit -- not PID gain or torque -- was capping how fast the
head could turn.

Co-Authored-By: Claude Sonnet 5 <noreply@anthropic.com>

File: urdf/sentry.urdf.xacro (robot description, xacro)
@@ -169,5 +169,5 @@
     <parent link="body"/>
     <child link="head"/>
-    <limit lower="-3.14159" upper="3.14159" effort="10" velocity="3"/>
+    <limit lower="-3.14159" upper="3.14159" effort="10" velocity="10"/>
   </joint>
   <joint name="lidarlink" type="fixed">
@@ -189,5 +189,5 @@
     <parent link="head"/>
     <child link="head_pitch"/>
-    <limit lower="-0.6" upper="0.6" effort="5" velocity="3"/>
+    <limit lower="-0.6" upper="0.6" effort="5" velocity="10"/>
   </joint>
   <joint name="cameralink" type="fixed">

Commit message: Tune headlink/headpitch PID to track the slider near-instantly
No kinematic direct-set mode exists in the installed gz-sim version
for JointPositionController (checked: no use_force_commands symbol in
the .so), so this can't be truly PID-free -- instead drop i_gain to 0
(no benefit for a disturbance-free instant setpoint, only adds lag),
raise p_gain/cmd_max and the joints' own effort limits so torque never
clips, leaving the velocity limit as the only real bottleneck. Given
the head's ~0.005kg mass this converges within about one physics step,
effectively indistinguishable from direct tracking.

Co-Authored-By: Claude Sonnet 5 <noreply@anthropic.com>

File: urdf/sentry.urdf.xacro (robot description, xacro)
@@ -169,5 +169,5 @@
     <parent link="body"/>
     <child link="head"/>
-    <limit lower="-3.14159" upper="3.14159" effort="10" velocity="10"/>
+    <limit lower="-3.14159" upper="3.14159" effort="200" velocity="10"/>
   </joint>
   <joint name="lidarlink" type="fixed">
@@ -189,5 +189,5 @@
     <parent link="head"/>
     <child link="head_pitch"/>
-    <limit lower="-0.6" upper="0.6" effort="5" velocity="10"/>
+    <limit lower="-0.6" upper="0.6" effort="200" velocity="10"/>
   </joint>
   <joint name="cameralink" type="fixed">
@@ -341,14 +341,24 @@
          impossible without overriding it here first. Hardcodes "sentry"
          since gz's topic templating doesn't reach into plugin params. -->
+    <!-- No kinematic "direct set" mode exists for this plugin in the
+         installed gz-sim version (checked: the .so exports no
+         use_force_commands symbol, unlike newer gz-sim releases), so this
+         stays PID-based, but tuned to converge within roughly one physics
+         step given headlink's tiny inertia: i_gain dropped to 0 (integral
+         term only added lag/overshoot, no benefit for a disturbance-free
+         instant setpoint), d_gain lowered accordingly since it no longer
+         needs to counteract windup, and cmd_max/effort (see the joint's
+         own limit above) raised well past what's needed so torque is
+         never the bottleneck, only the joint's velocity limit is. -->
     <plugin filename="ignition-gazebo-joint-position-controller-system" name="ignition::gazebo::systems::JointPositionController">
       <joint_name>headlink</joint_name>
       <topic>/model/sentry/joint/headlink/cmd_pos</topic>
-      <p_gain>50.0</p_gain>
-      <i_gain>0.1</i_gain>
-      <d_gain>1.0</d_gain>
-      <i_max>1</i_max>
-      <i_min>-1</i_min>
-      <cmd_max>50</cmd_max>
-      <cmd_min>-50</cmd_min>
+      <p_gain>300.0</p_gain>
+      <i_gain>0.0</i_gain>
+      <d_gain>0.5</d_gain>
+      <i_max>0</i_max>
+      <i_min>0</i_min>
+      <cmd_max>200</cmd_max>
+      <cmd_min>-200</cmd_min>
     </plugin>
     <!-- Same idea as headlink's controller above: publish a target angle
@@ -359,11 +369,11 @@
       <joint_name>headpitch</joint_name>
       <topic>/model/sentry/joint/headpitch/cmd_pos</topic>
-      <p_gain>50.0</p_gain>
-      <i_gain>0.1</i_gain>
-      <d_gain>1.0</d_gain>
-      <i_max>1</i_max>
-      <i_min>-1</i_min>
-      <cmd_max>50</cmd_max>
-      <cmd_min>-50</cmd_min>
+      <p_gain>300.0</p_gain>
+      <i_gain>0.0</i_gain>
+      <d_gain>0.5</d_gain>
+      <i_max>0</i_max>
+      <i_min>0</i_min>
+      <cmd_max>200</cmd_max>
+      <cmd_min>-200</cmd_min>
     </plugin>
     <!-- Lets the chassis actually be driven around in sim manually (e.g.

Commit message: Fix lidar self-visibility exclusion: use gazebo extension blocks, not inline tags
The previous fix put <visibility_flags> directly inside each link's
plain URDF <visual>, but URDF's schema doesn't define that element
there, so ros_gz_sim's spawn-time URDF->SDF conversion silently
dropped it -- confirmed by running the same conversion (`ign sdf -p`)
standalone and finding zero visibility_flags in the output. Moved it
into <gazebo reference="LINK"><visual> extension blocks instead
(alongside the existing gravity/sensor extensions this file already
uses for other SDF-only properties), and confirmed this time by
actually running the conversion: all 6 visuals now carry
visibility_flags=4294967294 (0xFFFFFFFE) and the lidar sensor carries
visibility_mask=1 in the resulting SDF.

Co-Authored-By: Claude Sonnet 5 <noreply@anthropic.com>

File: urdf/sentry.urdf.xacro (robot description, xacro)
@@ -16,13 +16,4 @@
         <color rgba="0.615686 0.811765 0.929412 1"/>
       </material>
-      <!-- Excluded from the lidar's own raycasting (see the lidar sensor's
-           visibility_mask=0x01 below), since the real RPLIDAR is mounted
-           with its scanning disk clear of the robot's own chassis. The
-           gpu_lidar sensor here is a rendering sensor with no physics
-           collision to fall back on (this model has none anywhere, by
-           design, see the root link comment further down), so without
-           this it also renders the robot's own visual meshes as scan
-           obstacles, which the real hardware never sees. -->
-      <visibility_flags>0xFFFFFFFE</visibility_flags>
     </visual>
   </link>
@@ -41,5 +32,4 @@
         <color rgba="0.615686 0.811765 0.929412 1"/>
       </material>
-      <visibility_flags>0xFFFFFFFE</visibility_flags>
     </visual>
   </link>
@@ -58,5 +48,4 @@
         <color rgba="0.615686 0.811765 0.929412 1"/>
       </material>
-      <visibility_flags>0xFFFFFFFE</visibility_flags>
     </visual>
   </link>
@@ -87,5 +76,4 @@
         <color rgba="0.1 0.1 0.1 1"/>
       </material>
-      <visibility_flags>0xFFFFFFFE</visibility_flags>
     </visual>
   </link>
@@ -104,5 +92,4 @@
         <color rgba="0.615686 0.811765 0.929412 1"/>
       </material>
-      <visibility_flags>0xFFFFFFFE</visibility_flags>
     </visual>
   </link>
@@ -121,5 +108,4 @@
         <color rgba="0.615686 0.811765 0.929412 1"/>
       </material>
-      <visibility_flags>0xFFFFFFFE</visibility_flags>
     </visual>
   </link>
@@ -228,9 +214,27 @@
     <gravity>false</gravity>
   </gazebo>
+  <!-- visibility_flags has to be injected here, as a <gazebo reference="...">
+       extension, rather than as a plain child of the link's own <visual> in
+       the URDF above: URDF's schema doesn't define that element inside
+       <visual>, so the URDF->SDF conversion ros_gz_sim's `create` runs at
+       spawn time silently drops it if it's written there (confirmed: `ign
+       sdf -p` on the xacro-expanded URDF showed zero visibility_flags
+       occurrences in its output when it was written inline). Matched
+       against visibility_mask=0x01 on the lidar sensor further down, so
+       (mask & flags) == 0 hides just these visuals from that one sensor
+       while leaving them visible to the GUI/RGBD camera and everything
+       else, which don't set visibility_mask and so keep sdformat's default
+       (0xFFFFFFFF); see the lidar sensor's own comment below for why. -->
   <gazebo reference="body">
     <gravity>false</gravity>
+    <visual>
+      <visibility_flags>0xFFFFFFFE</visibility_flags>
+    </visual>
   </gazebo>
   <gazebo reference="head">
     <gravity>false</gravity>
+    <visual>
+      <visibility_flags>0xFFFFFFFE</visibility_flags>
+    </visual>
   </gazebo>
   <gazebo reference="head_pitch">
@@ -239,12 +243,24 @@
   <gazebo reference="camera">
     <gravity>false</gravity>
+    <visual>
+      <visibility_flags>0xFFFFFFFE</visibility_flags>
+    </visual>
   </gazebo>
   <gazebo reference="odowheel">
     <gravity>false</gravity>
+    <visual>
+      <visibility_flags>0xFFFFFFFE</visibility_flags>
+    </visual>
   </gazebo>
   <gazebo reference="odowheel_1">
     <gravity>false</gravity>
+    <visual>
+      <visibility_flags>0xFFFFFFFE</visibility_flags>
+    </visual>
   </gazebo>
   <gazebo reference="lidar">
+    <visual>
+      <visibility_flags>0xFFFFFFFE</visibility_flags>
+    </visual>
     <sensor name="lidar" type="gpu_lidar">
       <always_on>true</always_on>

Commit message: Narrow lidar self-exclusion to just its own housing, not the whole body
Excluding body/head/camera/odowheel from the lidar's visibility made
the lidar see straight through its own head at every bearing, even
where the head is genuinely between the sensor and the world -- real
hardware's head really does obstruct part of the lidar's field of view
at whatever bearing it currently sits at (that's the whole reason
sim/head_sweep.py exists, to sweep that real blind wedge around).
Narrowed the exclusion to just the lidar's own housing mesh, which
wraps the sensor's exact origin and was the actual source of the
spurious near-zero-range self-hits; everything else keeps physically
occluding the beam like it should.

Co-Authored-By: Claude Sonnet 5 <noreply@anthropic.com>

File: urdf/sentry.urdf.xacro (robot description, xacro)
@@ -214,27 +214,9 @@
     <gravity>false</gravity>
   </gazebo>
-  <!-- visibility_flags has to be injected here, as a <gazebo reference="...">
-       extension, rather than as a plain child of the link's own <visual> in
-       the URDF above: URDF's schema doesn't define that element inside
-       <visual>, so the URDF->SDF conversion ros_gz_sim's `create` runs at
-       spawn time silently drops it if it's written there (confirmed: `ign
-       sdf -p` on the xacro-expanded URDF showed zero visibility_flags
-       occurrences in its output when it was written inline). Matched
-       against visibility_mask=0x01 on the lidar sensor further down, so
-       (mask & flags) == 0 hides just these visuals from that one sensor
-       while leaving them visible to the GUI/RGBD camera and everything
-       else, which don't set visibility_mask and so keep sdformat's default
-       (0xFFFFFFFF); see the lidar sensor's own comment below for why. -->
   <gazebo reference="body">
     <gravity>false</gravity>
-    <visual>
-      <visibility_flags>0xFFFFFFFE</visibility_flags>
-    </visual>
   </gazebo>
   <gazebo reference="head">
     <gravity>false</gravity>
-    <visual>
-      <visibility_flags>0xFFFFFFFE</visibility_flags>
-    </visual>
   </gazebo>
   <gazebo reference="head_pitch">
@@ -243,20 +225,31 @@
   <gazebo reference="camera">
     <gravity>false</gravity>
-    <visual>
-      <visibility_flags>0xFFFFFFFE</visibility_flags>
-    </visual>
   </gazebo>
   <gazebo reference="odowheel">
     <gravity>false</gravity>
-    <visual>
-      <visibility_flags>0xFFFFFFFE</visibility_flags>
-    </visual>
   </gazebo>
   <gazebo reference="odowheel_1">
     <gravity>false</gravity>
-    <visual>
-      <visibility_flags>0xFFFFFFFE</visibility_flags>
-    </visual>
-  </gazebo>
+  </gazebo>
+  <!-- Excludes only the lidar's own housing mesh from its own scan (via
+       visibility_mask=0x01 on the sensor below, matched against
+       visibility_flags=0xFFFFFFFE here so mask & flags evaluates to
+       zero). That mesh wraps the sensor's exact origin, so gpu_lidar (a
+       rendering sensor with no physics collision to fall back on; this
+       model has none anywhere, by design) was reporting spurious
+       near-zero-range self-hits against it. This intentionally does NOT
+       extend to body/head/camera/odowheel: head, in particular, genuinely
+       obstructs part of the lidar's real field of view at whatever
+       bearing it currently sits at (matching real hardware, see
+       sim/head_sweep.py's docstring, which sweeps the head specifically
+       to move that real blind wedge around over time) and should keep
+       physically blocking/occluding the beam there, not become invisible
+       to it. Injected via a <gazebo reference="..."> extension rather than
+       as a plain child of the link's own <visual> in the URDF above:
+       URDF's schema doesn't define visibility_flags inside <visual>, so
+       the URDF->SDF conversion ros_gz_sim's `create` runs at spawn time
+       silently drops it if it's written there (confirmed: `ign sdf -p` on
+       the xacro-expanded URDF showed zero visibility_flags occurrences in
+       its output when it was written inline). -->
   <gazebo reference="lidar">
     <visual>

Commit message: Revert lidar visibility_mask/flags hack; self-occlusion now a sentry_pkg filter
gz-sim's visibility_mask/visibility_flags could only ever be
all-or-nothing per visual: either fully invisible to the lidar (seeing
straight through the head even where it should genuinely occlude) or
fully visible (reporting the head's own mesh as a false self-hit) --
no way to express "block the beam here without counting it as a
detection." Removed entirely in favor of sentry_pkg's new
lidar_self_filter node, a software filter that blanks a fixed angular
sector of /scan_raw and republishes /scan; that works for real
hardware too, which has no rendering tricks available at all.

scan_bridge now remaps gz's /scan to ROS /scan_raw so
lidar_self_filter (launched from sentry_pkg/launch/auto.launch.py) is
the only thing publishing the final /scan, matching real hardware's
sllidar_node -> scan_raw -> lidar_self_filter -> scan pipeline.

Co-Authored-By: Claude Sonnet 5 <noreply@anthropic.com>

File: urdf/sentry.urdf.xacro (robot description, xacro)
@@ -232,28 +232,20 @@
     <gravity>false</gravity>
   </gazebo>
-  <!-- Excludes only the lidar's own housing mesh from its own scan (via
-       visibility_mask=0x01 on the sensor below, matched against
-       visibility_flags=0xFFFFFFFE here so mask & flags evaluates to
-       zero). That mesh wraps the sensor's exact origin, so gpu_lidar (a
-       rendering sensor with no physics collision to fall back on; this
-       model has none anywhere, by design) was reporting spurious
-       near-zero-range self-hits against it. This intentionally does NOT
-       extend to body/head/camera/odowheel: head, in particular, genuinely
-       obstructs part of the lidar's real field of view at whatever
-       bearing it currently sits at (matching real hardware, see
-       sim/head_sweep.py's docstring, which sweeps the head specifically
-       to move that real blind wedge around over time) and should keep
-       physically blocking/occluding the beam there, not become invisible
-       to it. Injected via a <gazebo reference="..."> extension rather than
-       as a plain child of the link's own <visual> in the URDF above:
-       URDF's schema doesn't define visibility_flags inside <visual>, so
-       the URDF->SDF conversion ros_gz_sim's `create` runs at spawn time
-       silently drops it if it's written there (confirmed: `ign sdf -p` on
-       the xacro-expanded URDF showed zero visibility_flags occurrences in
-       its output when it was written inline). -->
+  <!-- Self-occlusion (the lidar's own housing mesh, and the head's real
+       partial blocking of its own field of view at whatever bearing it
+       currently sits at, see sim/head_sweep.py's docstring) used to be
+       modeled here via gz-sim's visibility_mask/visibility_flags, but that
+       approach was all-or-nothing per visual: either a visual is fully
+       invisible to the lidar (so it also sees straight through the head
+       even where it should genuinely occlude) or fully visible (so it
+       reports the head's own mesh as a false self-hit), with no way to
+       express "block the beam here without counting it as a detection".
+       Removed in favor of sentry_pkg's lidar_self_filter node, a software
+       filter that blanks a fixed angular sector of /scan_raw; see that
+       node's docstring for why a fixed sector is valid here (the lidar
+       rotates rigidly with the head) and for the actual measured sector.
+       That approach also works for real hardware, which has no rendering
+       tricks available at all. -->
   <gazebo reference="lidar">
-    <visual>
-      <visibility_flags>0xFFFFFFFE</visibility_flags>
-    </visual>
     <sensor name="lidar" type="gpu_lidar">
       <always_on>true</always_on>
@@ -282,12 +274,4 @@
           <stddev>0.03</stddev>
         </noise>
-        <!-- Matched against visibility_flags=0xFFFFFFFE on the robot's own
-             visuals above (bit 0 cleared there): (mask & flags) == 0 for
-             those, so this lidar no longer scans its own body/head/camera/
-             odowheels, matching real hardware, which never sees itself.
-             Nothing else in the world sets visibility_flags, so everything
-             else keeps the sdformat default (0xFFFFFFFF) and stays fully
-             visible to this sensor. -->
-        <visibility_mask>0x01</visibility_mask>
       </lidar>
     </sensor>

Commit message: Add cv_head_aim: drive sim head from CV detections, fix headlink limit
New node converts sentry_pkg's /cv/target into /head_pan_cmd +
/head_pitch_cmd so the head actually tracks CV detections in sim,
instead of only head_sweep.py's unwired placeholder sweep.

Two bugs found and fixed against the live closed loop: corrections
reacting to every /cv/target arrival (up to 60Hz) raced the setpoint
ahead of what the physical joint could follow, causing a continuous
spin rather than convergence -- moved to a fixed-rate control timer
decoupled from detection rate. sign_pitch was also inverted, driving
pitch into positive feedback pegged at its -0.6 limit ("looking up");
fixed and verified converging to the analytically-expected angle.

Also fixes sentry.urdf.xacro's headlink joint, which was stale
type="revolute" with a +-pi <limit> -- real hardware's gimbal spins
freely, and sentry_pkg's own copy of this file already had it right
as type="continuous".

Co-Authored-By: Claude Sonnet 5 <noreply@anthropic.com>

File: urdf/sentry.urdf.xacro (robot description, xacro)
@@ -164,10 +164,9 @@
     <child link="body"/>
   </joint>
-  <joint name="headlink" type="revolute">
+  <joint name="headlink" type="continuous">
     <origin xyz="-2.54975e-18 5.65558e-17 0.252215" rpy="0 -0 3.14159"/>
     <axis xyz="0 0 -1"/>
     <parent link="body"/>
     <child link="head"/>
-    <limit lower="-3.14159" upper="3.14159" effort="200" velocity="10"/>
   </joint>
   <joint name="lidarlink" type="fixed">

Commit message: sentry.urdf.xacro: 9 kg chassis, head at 1/4 mass with matching PID
The sim robot weighed ~0.18 kg, 0.08 kg of it head, with the 72 g camera
0.1 m off the yaw axis. root floats free (no gravity, no collision), so
conserved momentum swung the chassis ~4-5 cm opposite every head turn.
root is now 8.9 kg (the real robot is ~9 kg; it is velocity-driven, so
driving is unchanged). Every head link's mass and inertia is scaled to 1/4,
and both head JointPositionControllers' p_gain, d_gain and cmd limits by
the same 1/4, which leaves the head's response unchanged.

Measured over a stationary + 0.5 m/s shot-hit run with the head sweeping
1.35 rad: chassis offset from spawn 0.0 mm. Stationary hit rate 90-96%,
0.5 m/s lead-on 80% vs lead-off 12%.

Co-Authored-By: Claude Opus 5 (1M context) <noreply@anthropic.com>

File: urdf/sentry.urdf.xacro (robot description, xacro)
@@ -20,7 +20,7 @@
   <link name="head">
     <inertial>
-      <mass value="0.00414744"/>
+      <mass value="0.00103686"/>
       <origin xyz="-0.00211769 -0.00164536 0.0741316" rpy="0 -0 1.18195"/>
-      <inertia ixx="2.08028e-05" ixy="-3.50322e-06" ixz="-4.24357e-08" iyy="1.60288e-05" iyz="-3.29709e-08" izz="2.21034e-05"/>
+      <inertia ixx="5.2007e-06" ixy="-8.75805e-07" ixz="-1.06089e-08" iyy="4.0072e-06" iyz="-8.24272e-09" izz="5.52585e-06"/>
     </inertial>
     <visual>
@@ -36,7 +36,7 @@
   <link name="lidar">
     <inertial>
-      <mass value="0.00018588"/>
+      <mass value="4.647e-05"/>
       <origin xyz="2.43997e-19 -6.96211e-19 0.02065" rpy="0 -0 1.90788"/>
-      <inertia ixx="9.29949e-08" ixy="0" ixz="0" iyy="9.29949e-08" iyz="0" izz="1.33148e-07"/>
+      <inertia ixx="2.32487e-08" ixy="0" ixz="0" iyy="2.32487e-08" iyz="0" izz="3.3287e-08"/>
     </inertial>
     <visual>
@@ -55,7 +55,7 @@
   <link name="head_pitch">
     <inertial>
-      <mass value="0.005"/>
+      <mass value="0.00125"/>
       <origin xyz="0 0 0" rpy="0 0 0"/>
-      <inertia ixx="1e-06" ixy="0" ixz="0" iyy="1e-06" iyz="0" izz="1e-06"/>
+      <inertia ixx="2.5e-07" ixy="0" ixz="0" iyy="2.5e-07" iyz="0" izz="2.5e-07"/>
     </inertial>
   </link>
@@ -64,7 +64,7 @@
   <link name="camera">
     <inertial>
-      <mass value="0.072"/>
+      <mass value="0.018"/>
       <origin xyz="0 0 0" rpy="0 0 0"/>
-      <inertia ixx="1.05e-05" ixy="0" ixz="0" iyy="5.4e-05" iyz="0" izz="5.4e-05"/>
+      <inertia ixx="2.625e-06" ixy="0" ixz="0" iyy="1.35e-05" iyz="0" izz="1.35e-05"/>
     </inertial>
     <visual>
@@ -153,5 +153,6 @@
   <link name="root">
     <inertial>
-      <mass value="0.0507536"/>
+      <!-- ~9 kg, the real robot's mass, so the head's reaction barely moves it. -->
+      <mass value="8.9"/>
       <origin xyz="-2.33205e-05 -3.02404e-05 0.160359" rpy="0 -0 0"/>
       <inertia ixx="2.26416" ixy="0" ixz="0" iyy="2.26416" iyz="0" izz="2.26416"/>
@@ -385,11 +386,11 @@
       <joint_name>headlink</joint_name>
       <topic>/model/sentry/joint/headlink/cmd_pos</topic>
-      <p_gain>300.0</p_gain>
+      <p_gain>75</p_gain>
       <i_gain>0.0</i_gain>
-      <d_gain>0.5</d_gain>
+      <d_gain>0.125</d_gain>
       <i_max>0</i_max>
       <i_min>0</i_min>
-      <cmd_max>200</cmd_max>
-      <cmd_min>-200</cmd_min>
+      <cmd_max>50</cmd_max>
+      <cmd_min>-50</cmd_min>
     </plugin>
     <!-- Same idea as headlink's controller above: publish a target angle
@@ -400,11 +401,11 @@
       <joint_name>headpitch</joint_name>
       <topic>/model/sentry/joint/headpitch/cmd_pos</topic>
-      <p_gain>300.0</p_gain>
+      <p_gain>75</p_gain>
       <i_gain>0.0</i_gain>
-      <d_gain>0.5</d_gain>
+      <d_gain>0.125</d_gain>
       <i_max>0</i_max>
       <i_min>0</i_min>
-      <cmd_max>200</cmd_max>
-      <cmd_min>-200</cmd_min>
+      <cmd_max>50</cmd_max>
+      <cmd_min>-50</cmd_min>
     </plugin>
     <!-- Lets the chassis actually be driven around in sim manually (e.g.
