Commit message: sentry.urdf.xacro: the lidar no longer scans its own model
visibility_flags=0xFFFFFFFE on every robot visual against the gpu_lidar's
visibility_mask=0x01, restoring the July approach that was reverted as
"all-or-nothing per visual". All-or-nothing is the right answer: the real
RPLIDAR's disk is clear of the chassis, and lidar_self_filter already
models the head's footprint in the one place that also runs on hardware.

Measured 2026-09-23 with the exclusion off: the head blanked 118-180 deg
of /scan_raw as -inf (self-hits inside range_min), plus a rear sector out
to -45 deg that moved with the head's pose -- 863 to 1613 of 3000 beams,
against the filter's 1.0 rad. A bare gpu_lidar at the same height in the
same world returns all 3000 beams at 2.22-7.17 m, so it was the robot,
not the world or the sensor. The sentry's own sensor now does too.

Every drift and shot-hit number recorded before today was measured on the
blanked scan.

Co-Authored-By: Claude Opus 5 (1M context) <noreply@anthropic.com>

File: urdf/sentry.urdf.xacro (robot description, xacro)
@@ -216,7 +216,13 @@
   <gazebo reference="body">
     <gravity>false</gravity>
+    <visual>
+      <visibility_flags>0xFFFFFFFE</visibility_flags>
+    </visual>
   </gazebo>
   <gazebo reference="head">
     <gravity>false</gravity>
+    <visual>
+      <visibility_flags>0xFFFFFFFE</visibility_flags>
+    </visual>
   </gazebo>
   <gazebo reference="head_pitch">
@@ -225,27 +231,29 @@
   <gazebo reference="camera">
     <gravity>false</gravity>
+    <visual>
+      <visibility_flags>0xFFFFFFFE</visibility_flags>
+    </visual>
   </gazebo>
   <gazebo reference="odowheel">
     <gravity>false</gravity>
+    <visual>
+      <visibility_flags>0xFFFFFFFE</visibility_flags>
+    </visual>
   </gazebo>
   <gazebo reference="odowheel_1">
     <gravity>false</gravity>
-  </gazebo>
-  <!-- Self-occlusion (the lidar's own housing mesh, and the head's real
-       partial blocking of its own field of view at whatever bearing it
-       currently sits at) used to be
-       modeled here via gz-sim's visibility_mask/visibility_flags, but that
-       approach was all-or-nothing per visual: either a visual is fully
-       invisible to the lidar (so it also sees straight through the head
-       even where it should genuinely occlude) or fully visible (so it
-       reports the head's own mesh as a false self-hit), with no way to
-       express "block the beam here without counting it as a detection".
-       Removed in favor of thornbots_pkg's lidar_self_filter node, a software
-       filter that blanks a fixed angular sector of /scan_raw; see that
-       node's docstring for why a fixed sector is valid here (the lidar
-       rotates rigidly with the head) and for the actual measured sector.
-       That approach also works for real hardware, which has no rendering
-       tricks available at all. -->
+    <visual>
+      <visibility_flags>0xFFFFFFFE</visibility_flags>
+    </visual>
+  </gazebo>
+  <!-- Every robot visual carries visibility_flags=0xFFFFFFFE against this
+       sensor's visibility_mask=0x01, so the lidar never scans its own
+       model; thornbots_pkg's lidar_self_filter is the only model of the
+       head's real blind sector, the same one hardware runs.
+       see README.md for design rationale -->
   <gazebo reference="lidar">
+    <visual>
+      <visibility_flags>0xFFFFFFFE</visibility_flags>
+    </visual>
     <sensor name="lidar" type="gpu_lidar">
       <always_on>true</always_on>
@@ -291,4 +299,8 @@
           <stddev>0.03</stddev>
         </noise>
+        <!-- (mask & flags) == 0 for the robot's own visuals, so it sees
+             none of them. Everything else keeps sdformat's default
+             0xFFFFFFFF and stays visible. -->
+        <visibility_mask>0x01</visibility_mask>
       </lidar>
     </sensor>

Commit message: Sim: headlink turns about +z, emulators report head_yaw CCW like the MCB
Matches thornbots_pkg's URDF (TF yaw == head_yaw). sentry_v2.urdf/.yaml/
simplify_urdf and the old sentry.urdf.xacro get axis +z; cv_head_aim_core
and bench_world's solve return +azimuth; cv_target_emulator FK axis +z;
mcb_emulator_node's turret yaw = chassis + joint; pose_emulator and
bench_world publish chassis_yaw/rate unnegated and head_yaw as the world yaw.
New test_yaw_joints_turn_counter_clockwise pins the axes.

Tests (isaac_ros_jazzy_container): test_cv_head_aim, test_urdf_constants,
test_shot_face, test/mcb, flake8: 61 passed, 2 failed in
test_mcb_bridge_pty.py (same 2 fail without this change: 0 CV_TARGET frames
read). bench_world.cpp passes g++ -fsyntax-only; the sim package can't be
built there (no gz-sim installed), and no bench or drift run was made.

Co-Authored-By: Claude Sonnet 5.5 <noreply@anthropic.com>

File: urdf/sentry.urdf.xacro (robot description, xacro)
@@ -168,5 +168,5 @@
   <joint name="headlink" type="continuous">
     <origin xyz="-2.54975e-18 5.65558e-17 0.252215" rpy="0 -0 3.14159"/>
-    <axis xyz="0 0 -1"/>
+    <axis xyz="0 0 1"/>
     <parent link="body"/>
     <child link="head"/>

File: urdf/sentry_v2/sentry_v2.urdf (robot description, URDF)
Before this commit: robot sentry_v2, 18 links, 17 joints
Joints:
- joint headlink: axis -0 -0 -1 -> 0 0 1
