Commit message: sentry_v2: armor_0..3 frames from the CAD
simplify_urdf.py finds each armor module's face part in the Onshape
export (armor.face_mesh) and emits a fixed link per face on root: origin
at the face centre, +x the outward normal, +y horizontal, with a box of
the face's size as visual and collision. E2E needs them: the detector
stand-in reads panel poses, depth needs something to see, and shots are
scored against the faces.

From the CAD: the faces sit on the diagonals, 45 deg + k x 90 deg from
the gun, 0.252 m out; armor_0/2 at 0.230 m and armor_1/3 at 0.136 m
(lower edges 94 mm apart, S126 allows 100); every normal 75.0 deg from
up (S122). The face is 135 x 125 mm, the Small Armor Module, the only
size in ARCC 2026.

The regen changed only the URDF text; the meshes came out different
bytes under the container's trimesh, so the committed ones stay. The
xacro colours the faces and hides them from the lidar; gz lumps them
into root with their collisions. test_urdf_constants.py pins
thornbots_pkg's copies and checks the S122 cant and S126 stagger.

Co-Authored-By: Claude Opus 5.5 (1M context) <noreply@anthropic.com>

File: urdf/sentry_v2.urdf.xacro (robot description, xacro)
@@ -28,4 +28,8 @@
   <xacro:body_visual link="head" rgb="0.75 0.08 0.08"/>
   <xacro:body_visual link="head_pitch" rgb="0.9 0.35 0.1"/>
+  <xacro:body_visual link="armor_0" rgb="0.85 0.85 0.85"/>
+  <xacro:body_visual link="armor_1" rgb="0.85 0.85 0.85"/>
+  <xacro:body_visual link="armor_2" rgb="0.85 0.85 0.85"/>
+  <xacro:body_visual link="armor_3" rgb="0.85 0.85 0.85"/>
   <!-- Corner i: a sprung carrier (spring rate and travel are placeholders in
        sentry_v2.yaml) and a sphere wheel with no friction, so wheels ride

File: urdf/sentry_v2/sentry_v2.urdf (robot description, URDF)
Before this commit: robot sentry_v2, 14 links, 13 joints
Links:
- added link armor_0; collision box size=0.00301404 0.135002 0.125002; visual box size=0.00301404 0.135002 0.125002
- added link armor_1; collision box size=0.00301404 0.135002 0.125002; visual box size=0.00301404 0.135002 0.125002
- added link armor_2; collision box size=0.00301404 0.135002 0.125002; visual box size=0.00301404 0.135002 0.125002
- added link armor_3; collision box size=0.00301404 0.135002 0.125002; visual box size=0.00301404 0.135002 0.125002
Joints:
- added joint armor_0link: type fixed, parent root, child armor_0, origin xyz=0.178162 0.178426 0.230361 rpy=0 -0.261856 0.785329
- added joint armor_1link: type fixed, parent root, child armor_1, origin xyz=-0.177935 0.177863 0.135661 rpy=0 -0.261856 2.35613
- added joint armor_2link: type fixed, parent root, child armor_2, origin xyz=-0.178505 -0.178235 0.230361 rpy=0 -0.261856 -2.35627
- added joint armor_3link: type fixed, parent root, child armor_3, origin xyz=0.177593 -0.177673 0.135661 rpy=0 -0.261856 -0.785464

Commit message: Match test E1 stack: a ghost opponent, a detector stand-in, e2e.launch.py
e2e.launch.py brings up stage E1 of ../E2E_PLAN.md, unscored: sim with the
depth camera, our robot parked, one red sentry_v2 opponent on
target_driver's path, and the real chain from roi_depth_node through
target_selector, target_tracker and point_to_cv_target to cv_head_aim. A
ros2 topic pub puts us on blue.

- opponents.py: the opponent's URDF. No sensors, gravity or contacts,
  collision shapes as visuals (the CAD visuals took the depth camera's
  RTF from 1.10 to 0.61), every joint but the head's fixed, and the root
  hull drawn at 75% in x and y, since at full size it stood 3-7 cm proud
  of every panel (ray-cast from each panel along its normal).
- OpponentMover, a gz system on the opponent, sets its pose every physics
  step from the path bridged to /model/<name>/path. Tried first:
  VelocityControl, which moves only the robot sim.launch.py spawns (a
  later-spawned sentry_v2 took 1 m/s for 3 s and moved 5 mm), and
  set_pose from Python, which half the 4 ms steps skipped and the rest
  jumped up to 36 cm and 1.7 rad. Now every step moves 8 mm and 0.038
  rad at 2 m/s and 1.5 Hz.
- opponent_driver spawns it once the path starts.
- detector_standin, a component in camera_container, publishes
  /detections_output per depth frame, stamped with it: panels facing the
  camera within 72.5 deg, in the image, whose rendered depth agrees with
  truth within 0.1 m, in YOLO's 640x640 letterbox. Truth is gz's
  PosePublisher at 250 Hz, interpolated to the frame's stamp; panel and
  camera offsets come from robot_description. gtest for the geometry.
- sim.launch.py puts sim's lib dir on GZ_SIM_SYSTEM_PLUGIN_PATH; the
  xacro takes name:= so each copy's plugin topics are its own.

Checked on the Mac (2026-09-29), 2 m/s, 1.5 Hz opponent at ~3 m, ~40 s:
- the head follows the opponent the whole run;
- gz's TF for the head matches gz (best offset 0, 0.7 mrad), and the
  depth frame matches its stamp (floor depth, best offset 0, 4 mm);
- roi_depth_node's panel centres sit 2.7 cm (p50) from truth, with
  Realsense_ROI_Depth_Rectifier 9ad71e1.
Open, in AGENTS.md: scoring, odom drifting ~1 cm/s with our robot parked,
and the camera container losing a load_node reply at startup (1 of ~10
launches). Unit tier passes (42).

Co-Authored-By: Claude Opus 5.5 (1M context) <noreply@anthropic.com>

File: urdf/sentry_v2.urdf.xacro (robot description, xacro)
@@ -8,4 +8,10 @@
 <robot name="sentry" xmlns:xacro="http://www.ros.org/wiki/xacro">
   <xacro:arg name="camera" default="false"/>
+  <!-- The gz model name, so each copy's plugin topics are its own. -->
+  <xacro:arg name="name" default="sentry"/>
+  <!-- An opponent carries no sensors and has no gravity or contacts;
+       its OpponentMover system moves it. -->
+  <xacro:arg name="opponent" default="false"/>
+  <xacro:property name="name" value="$(arg name)"/>
   <xacro:include filename="$(find sim)/urdf/sentry_v2/sentry_v2.urdf"/>
   <!-- Colour (gz only; the generated URDF has no materials, so rviz draws it
@@ -62,4 +68,5 @@
        mode, 10 Hz and 800 beams over -pi..pi (rf2o assumes a zero-centred
        scan), 0.15-12 m, 0.01 m noise. -->
+  <xacro:unless value="$(arg opponent)">
   <gazebo reference="lidar">
     <sensor name="lidar" type="gpu_lidar">
@@ -92,4 +99,5 @@
     </sensor>
   </gazebo>
+  </xacro:unless>
   <!-- D435-like depth camera at 60 Hz, only with camera:=true. Depth alone:
        the detector stand-in reads truth, so nothing needs colour.
@@ -128,6 +136,21 @@
       <robot_base_frame>root</robot_base_frame>
       <publish_odom_tf>true</publish_odom_tf>
+      <tf_topic>/model/${name}/odom_tf</tf_topic>
       <dimensions>3</dimensions>
       <odom_publish_frequency>100</odom_publish_frequency>
+    </plugin>
+    <!-- The model's world pose and every link's pose in it, one stamped
+         Pose_V on /model/<name>/pose at 250 Hz: the match test's truth for
+         the camera and the panels (fixed-joint links like armor_i and
+         camera are lumped into their parents in gz). -->
+    <plugin filename="gz-sim-pose-publisher-system" name="gz::sim::systems::PosePublisher">
+      <publish_model_pose>true</publish_model_pose>
+      <publish_link_pose>true</publish_link_pose>
+      <publish_nested_model_pose>false</publish_nested_model_pose>
+      <publish_visual_pose>false</publish_visual_pose>
+      <publish_collision_pose>false</publish_collision_pose>
+      <publish_sensor_pose>false</publish_sensor_pose>
+      <use_pose_vector_msg>true</use_pose_vector_msg>
+      <update_frequency>250</update_frequency>
     </plugin>
     <!-- Every joint, so robot_state_publisher can place the wheels too. -->
@@ -138,5 +161,5 @@
     <plugin filename="gz-sim-joint-position-controller-system" name="gz::sim::systems::JointPositionController">
       <joint_name>headlink</joint_name>
-      <topic>/model/sentry/joint/headlink/cmd_pos</topic>
+      <topic>/model/${name}/joint/headlink/cmd_pos</topic>
       <p_gain>75</p_gain>
       <i_gain>0.0</i_gain>
@@ -149,5 +172,5 @@
     <plugin filename="gz-sim-joint-position-controller-system" name="gz::sim::systems::JointPositionController">
       <joint_name>headpitch</joint_name>
-      <topic>/model/sentry/joint/headpitch/cmd_pos</topic>
+      <topic>/model/${name}/joint/headpitch/cmd_pos</topic>
       <p_gain>75</p_gain>
       <i_gain>0.0</i_gain>
@@ -163,6 +186,37 @@
          about 1 cm/s but can't bounce. -->
     <plugin filename="gz-sim-velocity-control-system" name="gz::sim::systems::VelocityControl">
-      <topic>/model/sentry/cmd_vel</topic>
+      <topic>/model/${name}/cmd_vel</topic>
     </plugin>
   </gazebo>
+  <xacro:if value="$(arg opponent)">
+    <!-- No gravity and no contacts: an opponent only has to render (panels
+         hide behind the field and other robots in the depth image) and be
+         where its pose says; shots are scored geometrically. -->
+    <xacro:macro name="ghost" params="link">
+      <gazebo reference="${link}">
+        <gravity>false</gravity>
+        <collision>
+          <surface><contact><collide_bitmask>0x00</collide_bitmask></contact></surface>
+        </collision>
+      </gazebo>
+    </xacro:macro>
+    <!-- Rides target_driver's path, bridged to /model/<name>/path; root at
+         sentry_v2's settled height on its springs. -->
+    <gazebo>
+      <plugin filename="opponent_mover" name="sim::OpponentMover">
+        <z>-0.0115</z>
+      </plugin>
+    </gazebo>
+    <xacro:ghost link="root"/>
+    <xacro:ghost link="head"/>
+    <xacro:ghost link="head_pitch"/>
+    <xacro:ghost link="carrier_0"/>
+    <xacro:ghost link="carrier_1"/>
+    <xacro:ghost link="carrier_2"/>
+    <xacro:ghost link="carrier_3"/>
+    <xacro:ghost link="wheel_0"/>
+    <xacro:ghost link="wheel_1"/>
+    <xacro:ghost link="wheel_2"/>
+    <xacro:ghost link="wheel_3"/>
+  </xacro:if>
 </robot>
