Commit message: wip: opponent xacro

File: urdf/sentry_v2.urdf.xacro (robot description, xacro)
@@ -8,4 +8,12 @@
 <robot name="sentry" xmlns:xacro="http://www.ros.org/wiki/xacro">
   <xacro:arg name="camera" default="false"/>
+  <!-- The gz model name, so each copy's plugin topics are its own. -->
+  <xacro:arg name="name" default="sentry"/>
+  <!-- An opponent carries no sensors, and spins its chassis on
+       chassis_spin under a heading-fixed spin_base, since VelocityControl
+       takes a body-frame twist (a spinning chassis would swirl its path
+       between commands). -->
+  <xacro:arg name="opponent" default="false"/>
+  <xacro:property name="name" value="$(arg name)"/>
   <xacro:include filename="$(find sim)/urdf/sentry_v2/sentry_v2.urdf"/>
   <!-- Colour (gz only; the generated URDF has no materials, so rviz draws it
@@ -62,4 +70,5 @@
        mode, 10 Hz and 800 beams over -pi..pi (rf2o assumes a zero-centred
        scan), 0.15-12 m, 0.01 m noise. -->
+  <xacro:unless value="$(arg opponent)">
   <gazebo reference="lidar">
     <sensor name="lidar" type="gpu_lidar">
@@ -92,4 +101,5 @@
     </sensor>
   </gazebo>
+  </xacro:unless>
   <!-- D435-like depth camera at 60 Hz, only with camera:=true. Depth alone:
        the detector stand-in reads truth, so nothing needs colour.
@@ -131,4 +141,18 @@
       <odom_publish_frequency>100</odom_publish_frequency>
     </plugin>
+    <!-- The model's world pose and every link's pose in it, one stamped
+         Pose_V on /model/<name>/pose at 250 Hz: the match test's truth for
+         the camera and the panels (fixed-joint links like armor_i and
+         camera are lumped into their parents in gz). -->
+    <plugin filename="gz-sim-pose-publisher-system" name="gz::sim::systems::PosePublisher">
+      <publish_model_pose>true</publish_model_pose>
+      <publish_link_pose>true</publish_link_pose>
+      <publish_nested_model_pose>false</publish_nested_model_pose>
+      <publish_visual_pose>false</publish_visual_pose>
+      <publish_collision_pose>false</publish_collision_pose>
+      <publish_sensor_pose>false</publish_sensor_pose>
+      <use_pose_vector_msg>true</use_pose_vector_msg>
+      <update_frequency>250</update_frequency>
+    </plugin>
     <!-- Every joint, so robot_state_publisher can place the wheels too. -->
     <plugin filename="gz-sim-joint-state-publisher-system" name="gz::sim::systems::JointStatePublisher"/>
@@ -138,5 +162,5 @@
     <plugin filename="gz-sim-joint-position-controller-system" name="gz::sim::systems::JointPositionController">
       <joint_name>headlink</joint_name>
-      <topic>/model/sentry/joint/headlink/cmd_pos</topic>
+      <topic>/model/${name}/joint/headlink/cmd_pos</topic>
       <p_gain>75</p_gain>
       <i_gain>0.0</i_gain>
@@ -149,5 +173,5 @@
     <plugin filename="gz-sim-joint-position-controller-system" name="gz::sim::systems::JointPositionController">
       <joint_name>headpitch</joint_name>
-      <topic>/model/sentry/joint/headpitch/cmd_pos</topic>
+      <topic>/model/${name}/joint/headpitch/cmd_pos</topic>
       <p_gain>75</p_gain>
       <i_gain>0.0</i_gain>
@@ -163,6 +187,23 @@
          about 1 cm/s but can't bounce. -->
     <plugin filename="gz-sim-velocity-control-system" name="gz::sim::systems::VelocityControl">
-      <topic>/model/sentry/cmd_vel</topic>
+      <topic>/model/${name}/cmd_vel</topic>
     </plugin>
   </gazebo>
+  <xacro:if value="$(arg opponent)">
+    <link name="spin_base">
+      <inertial><mass value="1.0"/><inertia ixx="0.01" ixy="0" ixz="0" iyy="0.01" iyz="0" izz="0.01"/></inertial>
+    </link>
+    <joint name="chassis_spin" type="continuous">
+      <parent link="spin_base"/>
+      <child link="root"/>
+      <axis xyz="0 0 1"/>
+    </joint>
+    <gazebo>
+      <!-- Sets chassis_spin's velocity (rad/s) straight from the topic. -->
+      <plugin filename="gz-sim-joint-controller-system" name="gz::sim::systems::JointController">
+        <joint_name>chassis_spin</joint_name>
+        <topic>/model/${name}/joint/chassis_spin/cmd_vel</topic>
+      </plugin>
+    </gazebo>
+  </xacro:if>
 </robot>

Commit message: wip: ghost opponent

File: urdf/sentry_v2.urdf.xacro (robot description, xacro)
@@ -138,4 +138,5 @@
       <robot_base_frame>root</robot_base_frame>
       <publish_odom_tf>true</publish_odom_tf>
+      <tf_topic>/model/${name}/odom_tf</tf_topic>
       <dimensions>3</dimensions>
       <odom_publish_frequency>100</odom_publish_frequency>
@@ -191,4 +192,27 @@
   </gazebo>
   <xacro:if value="$(arg opponent)">
+    <!-- No gravity and no contacts: an opponent only has to render (panels
+         hide behind the field and other robots in the depth image) and be
+         where its pose says; shots are scored geometrically. -->
+    <xacro:macro name="ghost" params="link">
+      <gazebo reference="${link}">
+        <gravity>false</gravity>
+        <collision>
+          <surface><contact><collide_bitmask>0x00</collide_bitmask></contact></surface>
+        </collision>
+      </gazebo>
+    </xacro:macro>
+    <xacro:ghost link="spin_base"/>
+    <xacro:ghost link="root"/>
+    <xacro:ghost link="head"/>
+    <xacro:ghost link="head_pitch"/>
+    <xacro:ghost link="carrier_0"/>
+    <xacro:ghost link="carrier_1"/>
+    <xacro:ghost link="carrier_2"/>
+    <xacro:ghost link="carrier_3"/>
+    <xacro:ghost link="wheel_0"/>
+    <xacro:ghost link="wheel_1"/>
+    <xacro:ghost link="wheel_2"/>
+    <xacro:ghost link="wheel_3"/>
     <link name="spin_base">
       <inertial><mass value="1.0"/><inertia ixx="0.01" ixy="0" ixz="0" iyy="0.01" iyz="0" izz="0.01"/></inertial>

Commit message: wip: opponent spins by VelocityControl

File: urdf/sentry_v2.urdf.xacro (robot description, xacro)
@@ -10,8 +10,6 @@
   <!-- The gz model name, so each copy's plugin topics are its own. -->
   <xacro:arg name="name" default="sentry"/>
-  <!-- An opponent carries no sensors, and spins its chassis on
-       chassis_spin under a heading-fixed spin_base, since VelocityControl
-       takes a body-frame twist (a spinning chassis would swirl its path
-       between commands). -->
+  <!-- An opponent carries no sensors, has no gravity or contacts, and
+       spins through VelocityControl's angular z. -->
   <xacro:arg name="opponent" default="false"/>
   <xacro:property name="name" value="$(arg name)"/>
@@ -183,8 +181,9 @@
       <cmd_min>-50</cmd_min>
     </plugin>
-    <!-- Sets the chassis's full twist every step from /cmd_vel: planar
-         velocity as commanded, zero angular velocity (a hard yaw lock), and
-         zero vertical velocity, so the chassis settles onto its springs at
-         about 1 cm/s but can't bounce. -->
+    <!-- Sets the chassis's full twist every step from /cmd_vel, in the body
+         frame: planar velocity and yaw rate as commanded (our /cmd_vel has
+         zero yaw rate, a hard yaw lock; opponent_driver spins opponents),
+         and zero vertical velocity, so the chassis settles onto its springs
+         at about 1 cm/s but can't bounce. -->
     <plugin filename="gz-sim-velocity-control-system" name="gz::sim::systems::VelocityControl">
       <topic>/model/${name}/cmd_vel</topic>
@@ -203,5 +202,4 @@
       </gazebo>
     </xacro:macro>
-    <xacro:ghost link="spin_base"/>
     <xacro:ghost link="root"/>
     <xacro:ghost link="head"/>
@@ -215,19 +213,4 @@
     <xacro:ghost link="wheel_2"/>
     <xacro:ghost link="wheel_3"/>
-    <link name="spin_base">
-      <inertial><mass value="1.0"/><inertia ixx="0.01" ixy="0" ixz="0" iyy="0.01" iyz="0" izz="0.01"/></inertial>
-    </link>
-    <joint name="chassis_spin" type="continuous">
-      <parent link="spin_base"/>
-      <child link="root"/>
-      <axis xyz="0 0 1"/>
-    </joint>
-    <gazebo>
-      <!-- Sets chassis_spin's velocity (rad/s) straight from the topic. -->
-      <plugin filename="gz-sim-joint-controller-system" name="gz::sim::systems::JointController">
-        <joint_name>chassis_spin</joint_name>
-        <topic>/model/${name}/joint/chassis_spin/cmd_vel</topic>
-      </plugin>
-    </gazebo>
   </xacro:if>
 </robot>

Commit message: fix(sim): expose opponent models to lidar
Use opponent-specific render flags while preserving own-model exclusion and existing sensors, contact masks, and scoring gates.

Register seven host-capable xacro visibility and CAD-section checks. At z=0.355 m, the central CAD silhouette measures 0.1517-0.2521 m, median 0.2369 m; record the narrower top slice and rendered-hull limitations.

Validation: Python 3.12 pytest (7 passed), repository quality (205 files, zero diagnostics), actionlint, flake8, pydocstyle, and changed documentation link. Parent owns ROS/container integration validation; no container launched here.

File: urdf/sentry_v2.urdf.xacro (robot description, xacro)
@@ -22,8 +22,9 @@
   <xacro:property name="name" value="$(arg name)"/>
   <xacro:include filename="$(find sim)/urdf/sentry_v2/sentry_v2.urdf"/>
-  <!-- Colour (gz only; the generated URDF has no materials, so rviz draws it
-       grey), and hidden from the lidar: visibility_mask 0x01 below renders
-       none of the robot, and lidar_self_filter models the blind sector
-       instead, as on hardware. -->
+  <!-- Only our model is hidden from the lidar; opponent copies render with
+       the field's default flags. lidar_self_filter models our blind sector,
+       as on hardware. Colour is gz-only (the generated URDF has no material). -->
+  <xacro:property name="is_opponent" value="$(arg opponent)"/>
+  <xacro:property name="lidar_visibility" value="${'0xFFFFFFFF' if is_opponent else '0xFFFFFFFE'}"/>
   <xacro:macro name="body_visual" params="link rgb">
     <gazebo reference="${link}">
@@ -34,5 +35,5 @@
           <specular>0.3 0.3 0.3 1</specular>
         </material>
-        <visibility_flags>0xFFFFFFFE</visibility_flags>
+        <visibility_flags>${lidar_visibility}</visibility_flags>
       </visual>
     </gazebo>

Commit message: fix(model): align sentry simulation geometry with the new CAD
Import the team's 2026-10-26 low-resolution body/head meshes and hulls,
head/sensor/muzzle origins and armor faces. Rebase yaw -y to ROS head +x
and the exported 20-degree elevation to horizontal zero pitch. Update
geometry constants in simulation consumers; retain controller algorithms,
plugins, topics, dynamics, chassis collision, wheels and suspension.
Capture/restore the configured self-filter mask in scan_degraded rather
than restoring obsolete hardcoded angles. Pin lidar parity to robot TF.

CAD zip SHA256:
0841b0ca27e54125ad8d962edf78dad97ce76198bb9d3b7c69036974ba32adff
Head lidar FOV: (-0.105,-0.193326,0.101293), yaw -0.149533673 rad.
Pitch camera IR apex: (0.095699877,-0.011500052,0.055000043).
Pitch muzzle front bore: (0.1729764,0.00190269,0).
Yaw bearing clearance datum z=0.267503694; pitch z=0.136 above yaw.
The uneven exported wheel pose does not establish a settled ground plane.

Validation: build, xacro/check_urdf, quality checker and actionlint pass.
Before: parked12/12, drive1/1, drift9/10; parked_push rerun passes.
After: parked12/12, drive1/1, final drift10/10; native logs accepted.
Worst parked localization p95 grows 0.075829 to 0.112258 m in these runs.
Registered package tests:499, six reported failures (four GTest cases and
two wrappers): ArmorRules and three existing aiming tests. Supplied CAD
stagger is103.885mm versus100mm; the unchanged aiming solver assumes a
pitch-axis muzzle and fails with the new forward offset. Keep these gates
visible: resolving armor acceptance/aiming is outside this geometry task.

File: urdf/sentry_v2.urdf.xacro (robot description, xacro)
@@ -64,5 +64,5 @@
   <xacro:corner i="2"/>
   <xacro:corner i="3"/>
-  <!-- Where the shot leaves: on the pitch axis, between the flywheels.
+  <!-- Where the shot leaves: at the front bore centre of the 2026-10-26 CAD.
        thornbots_pkg's URDF carries the same frame. -->
   <link name="muzzle"/>
@@ -70,5 +70,5 @@
     <parent link="head_pitch"/>
     <child link="muzzle"/>
-    <origin xyz="0 0.1128 0" rpy="0 0 0"/>
+    <origin xyz="0.1729764 0.00190269 0" rpy="0 0 0"/>
   </joint>
   <!-- Same angle-compensated A2M8 grid as sentry.urdf.xacro;

File: urdf/sentry_v2/sentry_v2.urdf (robot description, URDF)
Before this commit: robot sentry_v2, 18 links, 17 joints
Joints:
- joint armor_0link: origin xyz=0.178162 0.178426 0.230361 rpy=0 -0.261856 0.785329 -> xyz=0.204139959 0.150682952 0.148603392 rpy=0 -0.261799339 0.635864487
- joint armor_1link: origin xyz=-0.177935 0.177863 0.135661 rpy=0 -0.261856 2.35613 -> xyz=-0.148299431 0.200910863 0.25248797 rpy=0 -0.261797504 2.206660314
- joint armor_2link: origin xyz=-0.178505 -0.178235 0.230361 rpy=0 -0.261856 -2.35627 -> xyz=-0.204139942 -0.150683009 0.148603318 rpy=0 -0.261796504 -2.505724829
- joint armor_3link: origin xyz=0.177593 -0.177673 0.135661 rpy=0 -0.261856 -0.785464 -> xyz=0.148299403 -0.200910883 0.252487973 rpy=0 -0.261799535 -0.934934345
- joint cameralink: origin xyz=0.0920381 0.0948673 0.0566588 -> xyz=0.095699877 -0.011500052 0.055000043 rpy=0 0 0
- joint headlink: origin xyz=-0.000171242 9.52126e-05 0.248293 -> xyz=0 0 0.267503694 rpy=0 0 0
- joint headpitch: origin xyz=-0.00760542 -0.100122 0.14235 -> xyz=0 0 0.136 rpy=0 0 0
- joint lidarlink: origin xyz=-0.119391 -0.18501 0.0968001 -> xyz=-0.105 -0.193326 0.101293 rpy=0 0 -0.149533673

Commit message: fix(model): keep muzzle aiming origin on the pitch axis
Carry the CAD lateral offset into the existing aiming-frame contract. Restore pitch-invariant FK geometry without changing the solver or its ray and round-trip acceptance tests. Validation: aiming cases pass; the unchanged S126 armor rule still fails for the supplied CAD.

File: urdf/sentry_v2.urdf.xacro (robot description, xacro)
@@ -64,5 +64,5 @@
   <xacro:corner i="2"/>
   <xacro:corner i="3"/>
-  <!-- Where the shot leaves: at the front bore centre of the 2026-10-26 CAD.
+  <!-- Aiming origin on the pitch axis, between the flywheels; CAD lateral offset.
        thornbots_pkg's URDF carries the same frame. -->
   <link name="muzzle"/>
@@ -70,5 +70,5 @@
     <parent link="head_pitch"/>
     <child link="muzzle"/>
-    <origin xyz="0.1729764 0.00190269 0" rpy="0 0 0"/>
+    <origin xyz="0 0.00190269 0" rpy="0 0 0"/>
   </joint>
   <!-- Same angle-compensated A2M8 grid as sentry.urdf.xacro;
