Commit message: fix(field): use the corrected field assembly export
Import the supplied corrected field mesh and URDF, restoring the bar near y=+3 m at lidar height. Preserve world placement, routes and physics; document the canonical map and scope prior measurements to the earlier export.

Validation: 18 host geometry, route and combat cases pass, including the new bar regression. All four ZIP entries match, Python 3.12 quality and actionlint pass. No ROS build or simulation run performed.

File: world/real_field_assmbly/urdf/real_field_assmbly.urdf (robot description, URDF)
Before this commit: robot real_field_assmbly, 3 links, 2 joints
Links:
- link field: mass 9.62235 -> 9.63797
