Commit message: fix(lidar): match the spawned sensor to the measured robot mount
Use the Oct 26 CAD translation and measured 0.5907 rad scan-zero yaw on sentry_v2's lidarlink, matching thornbots_pkg #32. Restore the measured -0.5585..1.0123 rad blind sector after degraded-scan trials. Extend the existing URDF consistency check to include xacro lidar defaults.

Isolated Jazzy agent container: build succeeds with two compile jobs; colcon test sim: 224 tests, zero errors/failures, 87 skips. Host Python 3.12 quality and actionlint pass. Robot evidence and integration results live in workspace docs/investigations/lidar-mount-2026-10-26.md. No physical robot run.

File: urdf/sentry_v2/sentry_v2.urdf (robot description, URDF)
Before this commit: robot sentry_v2, 18 links, 17 joints
Joints:
- joint lidarlink: origin xyz=-0.119391 -0.18501 0.0968001 -> xyz=-0.105 -0.193326 0.101293 rpy=0 0 0.5907

Commit message: fix(urdf): put the sentry_v2 camera frame on the D435's RGB lens
simplify_urdf adds sentry_v2.yaml sensor_offsets to a sensor's part
centre; camera gets +32.5 mm left of the cover centre, the RGB lens that
roi_depth_node deprojects from. The generated URDF is edited to the same
value (the export is not in the repo), as are the bench and emulator
copies. The sim's truth detector shared the old frame, so it never showed
the real robot's 32.5 mm rightward aim error.

colcon test sim + thornbots_pkg 432/432, 0 skipped; aiming bench 10/10;
estimation bench 12/12.

File: urdf/sentry_v2/sentry_v2.urdf (robot description, URDF)
Before this commit: robot sentry_v2, 18 links, 17 joints
Joints:
- joint cameralink: origin xyz=0.0920381 0.0948673 0.0566588 -> xyz=0.0920381 0.127367 0.0566588

Commit message: feat: move the sim lidar to the flipped mount
Match thornbots_pkg's flipped-lidar defaults: lidarlink is now
(-0.0056, -0.193326, 0.063707) m, yaw 2.579 rad. The sim sensor stays
z-up, which is what the hardware driver publishes with inverted:=true.
The head mesh still shows the upright lidar; the sensor ignores it.

Tests: sim + thornbots_pkg colcon test in an archlinux agent container,
480 tests, 0 failures, 90 skips (UrdfConstants.SimModel included).
Quality check and actionlint pass.

File: urdf/sentry_v2/sentry_v2.urdf (robot description, URDF)
Before this commit: robot sentry_v2, 18 links, 17 joints
Joints:
- joint lidarlink: origin xyz=-0.105 -0.193326 0.101293 rpy=0 0 0.5907 -> xyz=-0.0056 -0.193326 0.063707 rpy=0 0 2.579
